File: 自作キーボード/10key-test/bottom.kicad_pcb (KiCad board)
At the start: 2 copper layers, 94.8 x 74.4 mm, 4 parts

Commit message: na
Other:
- board size 94.8 x 74.4 mm -> 95.3 x 74.9 mm
Changed lines of the file:
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@@
     (pad "" thru_hole circle (at 0 0) (size 6.5 6.5) (drill 4.3) (layers "*.Cu" "*.Mask"))
   )
-  (gr_arc (start 203.761631 132.988738) (mid 203.351739 132.614143) (end 203.2 132.08)
-    (stroke (width 0.1) (type default)) (layer "Edge.Cuts"))
-  (gr_arc (start 120.904001 138.176) (mid 121.20158 137.45758) (end 121.92 137.160001)
-    (stroke (width 0.1) (type default)) (layer "Edge.Cuts"))
-  (gr_line (start 161.925 71.12) (end 161.29 71.12)
+  (gr_line (start 112.395 93.345) (end 112.395 69.215)
     (stroke (width 0.05) (type default)) (layer "Edge.Cuts"))
-  (gr_arc (start 199.136 70.104) (mid 206.162124 68.157876) (end 204.216 75.184)
-    (stroke (width 0.1) (type default)) (layer "Edge.Cuts"))
-  (gr_line (start 198.12 137.16) (end 121.92 137.16)
-    (stroke (width 0.1) (type default)) (layer "Edge.Cuts"))
-  (gr_arc (start 198.12 137.16) (mid 198.654143 137.311739) (end 199.028738 137.721631)
-    (stroke (width 0.1) (type default)) (layer "Edge.Cuts"))
-  (gr_line (start 203.2 76.2) (end 203.2 132.08)
-    (stroke (width 0.1) (type default)) (layer "Edge.Cuts"))
-  (gr_arc (start 199.136 70.104) (mid 198.83842 70.82242) (end 198.12 71.12)
-    (stroke (width 0.1) (type default)) (layer "Edge.Cuts"))
-  (gr_arc (start 120.904001 138.176) (mid 113.877876 140.122124) (end 115.824 133.095999)
-    (stroke (width 0.1) (type default)) (layer "Edge.Cuts"))
-  (gr_arc (start 203.2 76.2) (mid 203.49758 75.48158) (end 204.216 75.184)
-    (stroke (width 0.1) (type default)) (layer "Edge.Cuts"))
-  (gr_arc (start 153.67 71.12) (mid 157.48 67.31) (end 161.29 71.12)
+  (gr_arc (start 114.3 141.605) (mid 112.952962 141.047038) (end 112.395 139.7)
     (stroke (width 0.05) (type default)) (layer "Edge.Cuts"))
-  (gr_arc (start 203.761631 132.988738) (mid 206.176143 140.136143) (end 199.028738 137.721631)
-    (stroke (width 0.1) (type default)) (layer "Edge.Cuts"))
-  (gr_line (start 116.84 97.155) (end 116.84 73.66)
+  (gr_line (start 114.3 141.605) (end 205.74 141.605)
     (stroke (width 0.05) (type default)) (layer "Edge.Cuts"))
-  (gr_line (start 116.84 132.08) (end 116.84 97.155)
-    (stroke (width 0.1) (type default)) (layer "Edge.Cuts"))
-  (gr_line (start 119.38 71.12) (end 153.67 71.12)
+  (gr_line (start 157.48 66.675) (end 114.935 66.675)
     (stroke (width 0.05) (type default)) (layer "Edge.Cuts"))
-  (gr_line (start 198.12 71.12) (end 161.925 71.12)
-    (stroke (width 0.1) (type default)) (layer "Edge.Cuts"))
-  (gr_arc (start 116.84 73.66) (mid 117.583949 71.863949) (end 119.38 71.12)
+  (gr_arc (start 207.645 139.7) (mid 207.087038 141.047038) (end 205.74 141.605)
     (stroke (width 0.05) (type default)) (layer "Edge.Cuts"))
-  (gr_arc (start 116.84 132.08) (mid 116.54242 132.79842) (end 115.824 133.096)
-    (stroke (width 0.1) (type default)) (layer "Edge.Cuts"))
+  (gr_arc (start 205.74 66.675) (mid 207.087038 67.232962) (end 207.645 68.58)
+    (stroke (width 0.05) (type default)) (layer "Edge.Cuts"))
+  (gr_arc (start 112.395 69.215) (mid 113.138949 67.418949) (end 114.935 66.675)
+    (stroke (width 0.05) (type default)) (layer "Edge.Cuts"))
+  (gr_line (start 205.74 66.675) (end 157.48 66.675)
+    (stroke (width 0.05) (type default)) (layer "Edge.Cuts"))
+  (gr_line (start 207.645 68.58) (end 207.645 139.7)
+    (stroke (width 0.05) (type default)) (layer "Edge.Cuts"))
+  (gr_line (start 112.395 139.7) (end 112.395 93.345)
+    (stroke (width 0.05) (type default)) (layer "Edge.Cuts"))
 )
